Commit message: temp

File: src/melodic/myrobot_description/urdf/myrobot.urdf.xacro (robot description, xacro)
@@ -8,7 +8,6 @@
     </gazebo>
     <xacro:include filename="$(find denso_robot_descriptions)/vs087_description/vs087.urdf.xacro" />
-    <!-- <xacro:include filename="$(find franka_description)/robots/hand.xacro" /> -->
-    <xacro:include filename="$(find franka_description)/robots/panda_gazebo.xacro" />
-    <!-- <xacro:include filename="$(find franka_description)/robots/utils.xacro" /> -->
+    <xacro:include filename="$(find franka_description)/robots/common/utils.xacro" />
+    <xacro:include filename="$(find franka_description)/robots/common/franka_hand.xacro"/>
     <xacro:include filename="$(find myrobot_description)/urdf/camera/_d435.urdf.xacro" />
     <xacro:include filename="$(find myrobot_description)/urdf/utils.xacro" />
@@ -29,5 +28,5 @@
         <xacro:f_joint name="${prefix}_joint_arm_base" xyz="${xyz}" rpy="${rpy}" parent="${parent}" child="${prefix}_base_link" />
         <xacro:vs087 prefix="${prefix}" />
-        <xacro:hand arm_id="${prefix}_panda" connected_to="${prefix}_J6" />
+        <xacro:franka_hand arm_id="${prefix}_panda" connected_to="${prefix}_J6" safety_distance="0" xyz="0 0 0.2" />
         <!-- to add transmission to hand | TODO: unuse gazebo-joint-->
         <!-- <xacro:gazebo-joint joint="${prefix}_panda_finger_joint1" transmission="hardware_interface/EffortJointInterface" />
@@ -71,4 +70,6 @@
     <xacro:property name="sholder_sz" value="0.24" />
     <!-- //////////////////////////////////////////////////////////////////////////////////////////////////////////////////////////////////////////////////////////////// -->
+    <link name="world" />
+    <xacro:f_joint name="world_joint" parent="world" child="base_link" />
     <link name="base_link" />
     <!-- cart -->
