Commit message: fix scoring and gazebo situation

File: src/melodic/myrobot_description/urdf/soft_hand/model.xacro (robot description, xacro)
@@ -18,5 +18,5 @@
             <collision>
                 <geometry>
-                    <mesh filename="package://myrobot_description/urdf/soft_hand/0F_top_asm_soft_gripper_v1_reduced.stl" scale="0.001 0.001 0.001" />
+                    <mesh filename="package://myrobot_description/urdf/soft_hand/untitled.dae" scale="0.001 0.001 0.001" />
                 </geometry>
                 <origin xyz="0.0 0.0 0.138" rpy="${radians(90)} 0.0 0.0" />
